File: picoletta.kicad_pcb (KiCad board)
At the start: 2 copper layers, 0 parts

Commit message: wip
Parts:
- added C1: 0.1uf 0402, Capacitor_SMD:C_0402_1005Metric, F.Cu at (89.8, 122.4)
- added C10: 10uf 0402, Capacitor_SMD:C_0603_1608Metric, F.Cu at (99.0, 125.2)
- added C11: 10uf 0603, Capacitor_SMD:C_0603_1608Metric, F.Cu at (99.0, 127.7)
- added C12: 1uf 0402, Capacitor_SMD:C_0402_1005Metric, F.Cu at (92.7, 126.3)
- added C13: 100nf 0402, Capacitor_SMD:C_0402_1005Metric, F.Cu at (92.7, 128.3)
- added C14: 100nf 0402, Capacitor_SMD:C_0402_1005Metric, F.Cu at (92.7, 130.3)
- added C15: 100nf 0402, Capacitor_SMD:C_0402_1005Metric, F.Cu at (92.7, 132.2)
- added C16: 100nf 0402, Capacitor_SMD:C_0402_1005Metric, F.Cu at (95.6, 122.4)
- added C17: 100nf 0402, Capacitor_SMD:C_0402_1005Metric, F.Cu at (95.6, 124.4)
- added C18: 100nf 0402, Capacitor_SMD:C_0402_1005Metric, F.Cu at (95.6, 126.3)
- added C19: 100nf 0402, Capacitor_SMD:C_0402_1005Metric, F.Cu at (95.6, 128.3)
- added C2: 22pf 0402, Capacitor_SMD:C_0402_1005Metric, F.Cu at (89.8, 124.4)
- added C20: 100nf 0402, Capacitor_SMD:C_0402_1005Metric, F.Cu at (95.6, 130.3)
- added C3: 22pf 0402, Capacitor_SMD:C_0402_1005Metric, F.Cu at (89.8, 126.3)
- added C4: 100nf 0402, Capacitor_SMD:C_0402_1005Metric, F.Cu at (89.8, 128.3)
- added C5: 10uf 0603, Capacitor_SMD:C_0603_1608Metric, F.Cu at (99.0, 122.7)
- added C6: 100nf 0402, Capacitor_SMD:C_0402_1005Metric, F.Cu at (89.8, 130.3)
- added C7: 100nf 0402, Capacitor_SMD:C_0402_1005Metric, F.Cu at (89.8, 132.2)
- added C8: 1uf 0402, Capacitor_SMD:C_0402_1005Metric, F.Cu at (92.7, 122.4)
- added C9: 22pF, Capacitor_SMD:C_0402_1005Metric, F.Cu at (92.7, 124.4)
- added D1: 1N4002W, Diode_SMD:D_SOD-123, F.Cu at (91.3, 77.7)
- added D_ASTA1: 1N4148W, Diode_SMD:D_SOD-123, F.Cu at (91.3, 81.0)
- added D_DEL1: 1N4148W, Diode_SMD:D_SOD-123, F.Cu at (91.3, 84.4)
- added D_EIGHT1: 1N4148W, Diode_SMD:D_SOD-123, F.Cu at (91.3, 87.7)
- added D_ENTER1: 1N4148W, Diode_SMD:D_SOD-123, F.Cu at (91.3, 91.1)
- added D_FIVE1: 1N4148W, Diode_SMD:D_SOD-123, F.Cu at (91.3, 94.4)
- added D_FOUR1: 1N4148W, Diode_SMD:D_SOD-123, F.Cu at (91.3, 97.8)
- added D_MACRO1: 1N4148W, Diode_SMD:D_SOD-123, F.Cu at (91.3, 101.1)
- added D_MACRO2: 1N4148W, Diode_SMD:D_SOD-123, F.Cu at (97.1, 77.7)
- added D_MACRO3: 1N4148W, Diode_SMD:D_SOD-123, F.Cu at (97.1, 81.0)
- added D_MACRO4: 1N4148W, Diode_SMD:D_SOD-123, F.Cu at (97.1, 84.4)
- added D_MINUS1: 1N4148W, Diode_SMD:D_SOD-123, F.Cu at (97.1, 87.7)
- added D_NINE1: 1N4148W, Diode_SMD:D_SOD-123, F.Cu at (97.1, 91.1)
- added D_NUM1: 1N4148W, Diode_SMD:D_SOD-123, F.Cu at (97.1, 94.4)
- added D_ONE1: 1N4148W, Diode_SMD:D_SOD-123, F.Cu at (97.1, 97.8)
- added D_PLUS1: 1N4148W, Diode_SMD:D_SOD-123, F.Cu at (97.1, 101.1)
- added D_ROT1: 1N4148W, Diode_SMD:D_SOD-123, F.Cu at (102.9, 77.7)
- added D_SEVEN1: 1N4148W, Diode_SMD:D_SOD-123, F.Cu at (102.9, 81.0)
- added D_SIX1: 1N4148W, Diode_SMD:D_SOD-123, F.Cu at (102.9, 84.4)
- added D_SLASH1: 1N4148W, Diode_SMD:D_SOD-123, F.Cu at (102.9, 87.7)
- added D_THREE1: 1N4148W, Diode_SMD:D_SOD-123, F.Cu at (102.9, 91.1)
- added D_TWO1: 1N4148W, Diode_SMD:D_SOD-123, F.Cu at (102.9, 94.4)
- added D_ZERO1: 1N4148W, Diode_SMD:D_SOD-123, F.Cu at (102.9, 97.8)
- added F1: 0805L050WR, Fuse:Fuse_0805_2012Metric, F.Cu at (108.0, 100.7)
- added FLASH1: W25Q16JVUXIQ, PB_W25Q256JVEIQ_TR:SON127P800X600X80-9N, F.Cu at (80.3, 132.6)
- added GPIO25_LED1: LED_0402, LED_SMD:LED_0402_1005Metric, F.Cu at (112.5, 132.1)
- added GPIO25_RESISTOR1: 470 0402, Resistor_SMD:R_0402_1005Metric, F.Cu at (105.2, 103.8)
- added J1: TSA343G00-250J2, Button_Switch_SMD:SW_Push_SPST_NO_Alps_SKRK, F.Cu at (109.0, 87.5)
- added J2: Conn_01x20_Socket, Connector_PinSocket_2.54mm:PinSocket_1x20_P2.54mm_Horizontal, F.Cu at (86.1, 78.3)
- added L1: SWPA3015S2R2NT, JLC2KiCadLib:IND-SMD_L3.0-W3.0, F.Cu at (108.3, 96.7)
- added R1: 5.1K 0402, Resistor_SMD:R_0402_1005Metric, F.Cu at (105.2, 105.8)
- added R10: 680K, Resistor_SMD:R_0402_1005Metric, F.Cu at (108.1, 111.8)
- added R11: 150K, Resistor_SMD:R_0402_1005Metric, F.Cu at (108.1, 113.7)
- added R12: 27r 0402 resistor, Resistor_SMD:R_0402_1005Metric, F.Cu at (111.0, 103.8)
- added R13: 27r 0402 resistor, Resistor_SMD:R_0402_1005Metric, F.Cu at (111.0, 105.8)
- added R14: 200 0603, Resistor_SMD:R_0603_1608Metric, F.Cu at (99.0, 130.2)
- added R15: 1 0402, Resistor_SMD:R_0402_1005Metric, F.Cu at (111.0, 107.8)
- added R2: 5.1K 0402, Resistor_SMD:R_0402_1005Metric, F.Cu at (105.2, 107.8)
- added R3: 220 0402, Resistor_SMD:R_0402_1005Metric, F.Cu at (105.2, 109.8)
- added R4: 1K 0402, Resistor_SMD:R_0402_1005Metric, F.Cu at (105.2, 111.8)
- added R5: 5.6K 0402, Resistor_SMD:R_0402_1005Metric, F.Cu at (105.2, 113.7)
- added R6: 10K 0402, Resistor_SMD:R_0402_1005Metric, F.Cu at (108.1, 103.8)
- added R7: 10K 0402, Resistor_SMD:R_0402_1005Metric, F.Cu at (108.1, 105.8)
- added R8: 1K 0402, Resistor_SMD:R_0402_1005Metric, F.Cu at (108.1, 107.8)
- added R9: 100K 0402, Resistor_SMD:R_0402_1005Metric, F.Cu at (108.1, 109.8)
- added RSW1: TSA343G00-250J2, Button_Switch_SMD:SW_Push_SPST_NO_Alps_SKRK, F.Cu at (109.0, 92.0)
- added SW_ASTA1: SW_PUSH, BrownSugar pretty:CherryMX_Hotswap_via_1U, F.Cu at (24.6, 25.6)
- added SW_DEL1: SW_PUSH, BrownSugar pretty:CherryMX_Hotswap_via_1U, F.Cu at (24.6, 45.7)
- added SW_EIGHT1: SW_PUSH, BrownSugar pretty:CherryMX_Hotswap_via_1U, F.Cu at (24.6, 65.9)
- added SW_ENTER1: SW_PUSH, BrownSugar pretty:CherryMX_Hotswap_via_2U, F.Cu at (94.6, 25.6)
- added SW_FIVE1: SW_PUSH, BrownSugar pretty:CherryMX_Hotswap_via_1U, F.Cu at (24.6, 86.1)
- added SW_FOUR1: SW_PUSH, BrownSugar pretty:CherryMX_Hotswap_via_1U, F.Cu at (24.6, 106.2)
- added SW_MACRO1: SW_PUSH, BrownSugar pretty:CherryMX_Hotswap_via_1U, F.Cu at (24.6, 126.4)
- added SW_MACRO2: SW_PUSH, BrownSugar pretty:CherryMX_Hotswap_via_1U, F.Cu at (44.8, 25.6)
- added SW_MACRO3: SW_PUSH, BrownSugar pretty:CherryMX_Hotswap_via_1U, F.Cu at (44.8, 45.7)
- added SW_MACRO4: SW_PUSH, BrownSugar pretty:CherryMX_Hotswap_via_1U, F.Cu at (44.8, 65.9)
- added SW_MINUS1: SW_PUSH, BrownSugar pretty:CherryMX_Hotswap_via_1U, F.Cu at (44.8, 86.1)
- added SW_NINE1: SW_PUSH, BrownSugar pretty:CherryMX_Hotswap_via_1U, F.Cu at (44.8, 106.2)
- added SW_NUM1: SW_PUSH, BrownSugar pretty:CherryMX_Hotswap_via_1U, F.Cu at (44.8, 126.4)
- added SW_ONE1: SW_PUSH, BrownSugar pretty:CherryMX_Hotswap_via_1U, F.Cu at (65.0, 25.6)
- added SW_PLUS1: SW_PUSH, BrownSugar pretty:CherryMX_Hotswap_via_2U, F.Cu at (94.6, 45.7)
- added SW_ROT1: RotaryEncoder_Switch, BrownSugar pretty:RotaryEncoder_EC11-Switch, F.Cu at (96.0, 111.9)
- added SW_SEVEN1: SW_PUSH, BrownSugar pretty:CherryMX_Hotswap_via_1U, F.Cu at (65.0, 45.7)
- added SW_SIX1: SW_PUSH, BrownSugar pretty:CherryMX_Hotswap_via_1U, F.Cu at (65.0, 65.9)
- added SW_SLASH1: SW_PUSH, BrownSugar pretty:CherryMX_Hotswap_via_1U, F.Cu at (65.0, 86.1)
- added SW_THREE1: SW_PUSH, BrownSugar pretty:CherryMX_Hotswap_via_1U, F.Cu at (65.0, 106.2)
- added SW_TWO1: SW_PUSH, BrownSugar pretty:CherryMX_Hotswap_via_1U, F.Cu at (65.0, 126.4)
- added SW_ZERO1: SW_PUSH, BrownSugar pretty:CherryMX_Hotswap_via_2U, F.Cu at (94.6, 65.9)
- added U1: TD6810, JLC2KiCadLib:SOT-23-5_L3.0-W1.7-P0.95-LS2.8-BR, F.Cu at (103.3, 133.3)
- added U2: RP2040, PB_RP2040_minimal:RP2040-QFN-56, F.Cu at (110.4, 80.6)
- added USB1: TYPE-C-31-M-12, PB_HRO-TYPE-C31-M-12:HRO-TYPE-C-31-M-12, F.Cu at (106.3, 130.3)
- added Y1: 3225_4P, Crystal:Crystal_SMD_3225-4Pin_3.2x2.5mm, F.Cu at (108.2, 133.3)

Commit message: wip
Parts:
- removed GPIO25_LED1: LED_0402, LED_SMD:LED_0402_1005Metric
- removed GPIO25_RESISTOR1: 470 0402, Resistor_SMD:R_0402_1005Metric
- added LED1: RGBLED_WS2812B, BrownSugar pretty:RGBLED_WS2812B, F.Cu at (78.6, 79.0)
- added LED10: RGBLED_WS2812B, BrownSugar pretty:RGBLED_WS2812B, F.Cu at (86.3, 91.3)
- added LED11: RGBLED_WS2812B, BrownSugar pretty:RGBLED_WS2812B, F.Cu at (86.3, 97.4)
- added LED12: RGBLED_WS2812B, BrownSugar pretty:RGBLED_WS2812B, F.Cu at (86.3, 103.5)
- added LED13: RGBLED_WS2812B, BrownSugar pretty:RGBLED_WS2812B, F.Cu at (86.3, 109.6)
- added LED14: RGBLED_WS2812B, BrownSugar pretty:RGBLED_WS2812B, F.Cu at (86.3, 115.8)
- added LED15: RGBLED_WS2812B, BrownSugar pretty:RGBLED_WS2812B, F.Cu at (93.9, 79.0)
- added LED16: RGBLED_WS2812B, BrownSugar pretty:RGBLED_WS2812B, F.Cu at (93.9, 85.2)
- added LED17: RGBLED_WS2812B, BrownSugar pretty:RGBLED_WS2812B, F.Cu at (93.9, 91.3)
- added LED18: RGBLED_WS2812B, BrownSugar pretty:RGBLED_WS2812B, F.Cu at (93.9, 97.4)
- added LED19: RGBLED_WS2812B, BrownSugar pretty:RGBLED_WS2812B, F.Cu at (93.9, 103.5)
- added LED2: RGBLED_WS2812B, BrownSugar pretty:RGBLED_WS2812B, F.Cu at (78.6, 85.2)
- added LED20: RGBLED_WS2812B, BrownSugar pretty:RGBLED_WS2812B, F.Cu at (93.9, 109.6)
- added LED21: RGBLED_WS2812B, BrownSugar pretty:RGBLED_WS2812B, F.Cu at (93.9, 115.8)
- added LED3: RGBLED_WS2812B, BrownSugar pretty:RGBLED_WS2812B, F.Cu at (78.6, 91.3)
- added LED4: RGBLED_WS2812B, BrownSugar pretty:RGBLED_WS2812B, F.Cu at (78.6, 97.4)
- added LED5: RGBLED_WS2812B, BrownSugar pretty:RGBLED_WS2812B, F.Cu at (78.6, 103.5)
- added LED6: RGBLED_WS2812B, BrownSugar pretty:RGBLED_WS2812B, F.Cu at (78.6, 109.6)
- added LED7: RGBLED_WS2812B, BrownSugar pretty:RGBLED_WS2812B, F.Cu at (78.6, 115.8)
- added LED8: RGBLED_WS2812B, BrownSugar pretty:RGBLED_WS2812B, F.Cu at (86.3, 79.0)
- added LED9: RGBLED_WS2812B, BrownSugar pretty:RGBLED_WS2812B, F.Cu at (86.3, 85.2)
- J1, RSW1: value TSA343G00-250J2 -> 1-1825027-7; footprint Button_Switch_SMD:SW_Push_SPST_NO_Alps_SKRK -> JLC2KiCadLib:SW-TH_KH-6X6X4.3H-ZJ
- moved J2 72.1 mm to (125.2, 17.7)
- moved U2 48.2 mm to (88.3, 123.5)
- moved L1 37.9 mm to (91.5, 130.6)
- moved FLASH1 34.3 mm to (113.8, 125.2)
- moved R15 34.0 mm to (82.2, 125.8)
- moved R12 34.0 mm to (82.2, 121.8)
- moved R13 34.0 mm to (82.2, 123.8)
- moved R10 32.9 mm to (79.3, 127.8)
- moved R6 32.9 mm to (79.3, 119.8)
- moved R7 32.9 mm to (79.3, 121.8)
- moved R8 32.9 mm to (79.3, 123.8)
- moved R9 32.9 mm to (79.3, 125.8)
- moved R1 32.0 mm to (76.4, 119.8)
- moved R2 32.0 mm to (76.4, 121.8)
- moved R4 32.0 mm to (76.4, 125.8)
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Connections:
- J2 pad 17: GND -> /DOUT
- U2 pad 37: /GPIO25 -> /DIN
