File: picoletta.kicad_sch (KiCad schematic)
At the start: 99 parts, among them J1 TSA343G00-250J2, J2 Conn_01x16_Socket, J4 Conn_01x03_Male, U1 TD6810-ADJ, U2 RP2040, Y1 3225_4P

Commit message: wip
Parts:
- removed H1, H2, H3, H4: MountingHole, MountingHole:MountingHole_2.1mm, symbol Mechanical:MountingHole
- removed J2: Conn_01x16_Socket, symbol Connector:Conn_01x16_Socket
- removed J4: Conn_01x03_Male, Connector_PinHeader_2.54mm:PinHeader_1x03_P2.54mm_Vertical, symbol Connector_Generic:Conn_01x03
- removed L1: 2.2uH, Inductor_SMD:WPN252010UF2R2MT, symbol Device:L_Small
- removed TP1, TP2: TestPoint, EnvExtras:CustomTestPoint, symbol Connector:TestPoint
- removed U1: TD6810-ADJ, Package_TO_SOT_SMD:SOT-23-5, symbol Custom_components:TD6810-ADJ
- added J2: Conn_01x20_Socket, Connector_PinSocket_2.54mm:PinSocket_1x20_P2.54mm_Horizontal, symbol Connector:Conn_01x20_Socket
- added L1: SWPA3015S2R2NT, JLC2KiCadLib:IND-SMD_L3.0-W3.0, symbol JLC2KiCadLib_SWPA3015S2R2NT:SWPA3015S2R2NT
- added U1: TD6810, JLC2KiCadLib:SOT-23-5_L3.0-W1.7-P0.95-LS2.8-BR, symbol JLC2KiCadLib_ TD6810:TD6810
- FLASH1: footprint SON127P800X600X80-9N -> PB_W25Q256JVEIQ_TR:SON127P800X600X80-9N; LCSC (none) -> (none); MANUFACTURER Winbond Electronics Corp. -> (none)
- SW_ASTA1, SW_DEL1, SW_EIGHT1, SW_FIVE1, SW_FOUR1, SW_MACRO1, SW_MACRO2, SW_MACRO3, SW_MACRO4, SW_MINUS1, SW_NINE1, SW_NUM1, SW_ONE1, SW_SEVEN1, SW_SIX1, SW_SLASH1, SW_THREE1, SW_TWO1: footprint (none) -> BrownSugar pretty:CherryMX_Hotswap_via_1U
- SW_ENTER1, SW_PLUS1, SW_ZERO1: footprint (none) -> BrownSugar pretty:CherryMX_Hotswap_via_2U
- SW_ROT1: footprint (none) -> BrownSugar pretty:RotaryEncoder_EC11-Switch
- U2: footprint RP2040_minimal:RP2040-QFN-56 -> PB_RP2040_minimal:RP2040-QFN-56
Connections:
- net +3V3: now also L1.2
- net 3V3_EN: now also U1.1 (RUN)
- net GND: now also J2.17 (Pin_17), J2.18 (Pin_18), U1.2 (GND)
- net GPIO12: now also J2.1 (Pin_1)
- net GPIO13: now also J2.2 (Pin_2)
- net GPIO14: now also J2.3 (Pin_3)
- net GPIO15: now also J2.4 (Pin_4)
- net GPIO16: now also J2.5 (Pin_5)
- net GPIO17: now also J2.6 (Pin_6)
- net GPIO18: now also J2.7 (Pin_7)
- net GPIO19: now also J2.8 (Pin_8)
- net GPIO20: now also J2.9 (Pin_9)
- net GPIO21: now also J2.10 (Pin_10)
- net GPIO22: now also J2.11 (Pin_11)
- net GPIO23: now also J2.12 (Pin_12)
- net GPIO26_ADC0: now also J2.13 (Pin_13)
- net GPIO27_ADC1: now also J2.14 (Pin_14)
- net GPIO28_ADC2: now also J2.15 (Pin_15)
- net GPIO29_ADC3: now also J2.16 (Pin_16)
- net SWCLK: now also J2.20 (Pin_20)
- net SWD: now also J2.19 (Pin_19)
- net at C9.1, R10.2, R11.2: now also U1.5 (VFB/VOUT)
- net at C5.1, F1.1: now also U1.4 (VIN)
- new net: L1.1, U1.3 (SW)
Other:
- note removed: "Test points"
- moved on the sheet: C11, C13, C9, R10, R11, R9

Commit message: wip
Parts:
- removed GPIO25_LED1: LED_0402, LED_SMD:LED_0402_1005Metric, symbol Device:LED
- removed GPIO25_RESISTOR1: 470 0402, Resistor_SMD:R_0402_1005Metric, symbol Device:R
- added LED1: RGBLED_WS2812B, BrownSugar pretty:RGBLED_SK6812MINI-E, symbol BrownSugar:RGBLED_WS2812B
- added LED10, LED11, LED12, LED13, LED14, LED15, LED16, LED17, LED18, LED19, LED2, LED20, LED21, LED3, LED4, LED5, LED6, LED7, LED8, LED9: RGBLED_WS2812B, BrownSugar pretty:RGBLED_WS2812B, symbol BrownSugar:RGBLED_WS2812B
- J1, RSW1: value TSA343G00-250J2 -> 1-1825027-7; footprint Button_Switch_SMD:SW_Push_SPST_NO_Alps_SKRK -> JLC2KiCadLib:SW-TH_KH-6X6X4.3H-ZJ; symbol Switch:SW_Push -> JLC2KiCadLib_1-1825027-7:1-1825027-7; LCSC (none) -> C592923
Connections:
- net GND: now also LED1.3 (GND), LED10.3 (GND), LED11.3 (GND), LED12.3 (GND), LED13.3 (GND), LED14.3 (GND), LED15.3 (GND), LED16.3 (GND), LED17.3 (GND), LED18.3 (GND), LED19.3 (GND), LED2.3 (GND), LED20.3 (GND), LED21.3 (GND), LED3.3 (GND), LED4.3 (GND), LED5.3 (GND), LED6.3 (GND), LED7.3 (GND), LED8.3 (GND), LED9.3 (GND); no longer J2.17 (Pin_17)
- net VBUS: now also LED1.1 (VDD), LED10.1 (VDD), LED11.1 (VDD), LED12.1 (VDD), LED13.1 (VDD), LED14.1 (VDD), LED15.1 (VDD), LED16.1 (VDD), LED17.1 (VDD), LED18.1 (VDD), LED19.1 (VDD), LED2.1 (VDD), LED20.1 (VDD), LED21.1 (VDD), LED3.1 (VDD), LED4.1 (VDD), LED5.1 (VDD), LED6.1 (VDD), LED7.1 (VDD), LED8.1 (VDD), LED9.1 (VDD)
- net GPIO25 renamed DIN
- net DIN: now also LED1.4 (DIN)
- new net: LED1.2 (DOUT), LED2.4 (DIN)
- new net: LED11.2 (DOUT), LED12.4 (DIN)
- new net: LED10.2 (DOUT), LED11.4 (DIN)
- new net: LED10.4 (DIN), LED9.2 (DOUT)
- new net: LED8.2 (DOUT), LED9.4 (DIN)
- new net: LED16.2 (DOUT), LED17.4 (DIN)
- new net: LED15.2 (DOUT), LED16.4 (DIN)
- new net: LED3.2 (DOUT), LED4.4 (DIN)
- new net: LED2.2 (DOUT), LED3.4 (DIN)
- new net: LED4.2 (DOUT), LED5.4 (DIN)
- new net: LED5.2 (DOUT), LED6.4 (DIN)
- new net: LED14.2 (DOUT), LED15.4 (DIN)
- new net: LED13.2 (DOUT), LED14.4 (DIN)
- new net: LED7.2 (DOUT), LED8.4 (DIN)
- new net: LED6.2 (DOUT), LED7.4 (DIN)
- new net: LED17.2 (DOUT), LED18.4 (DIN)
- new net: LED19.2 (DOUT), LED20.4 (DIN)
- new net: LED18.2 (DOUT), LED19.4 (DIN)
- new net: LED20.2 (DOUT), LED21.4 (DIN)
- new net: LED12.2 (DOUT), LED13.4 (DIN)
- new net DOUT: J2.17 (Pin_17), LED21.2 (DOUT)
- no-connect marks 2 -> 6
Other:
- note removed: "LEDs"
- moved on the sheet: C2, C3, C5, R8, Y1
